File: Hardware/Qwiic_IoT_Security_ATECC508A.brd (EAGLE design)
At the start: 25.4 x 25.4 mm, 37 parts, among them J1 QWIIC, J2 QWIIC, J3 PTH, U1 ATECC508A

Commit message: rotated LED jumper bPlace label so it reads upright
Parts:
- moved U$1 4.65 mm to (22.5, 9.19), turned to 0 degrees
Changed lines of the file:
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@@
 <grid distance="0.05" unitdist="inch" unit="inch" style="lines" multiple="1" display="yes" altdistance="0.001" altunitdist="inch" altunit="inch"/>
 <layers>
-<layer number="1" name="Top" color="4" fill="1" visible="yes" active="yes"/>
+<layer number="1" name="Top" color="4" fill="1" visible="no" active="yes"/>
 <layer number="16" name="Bottom" color="1" fill="1" visible="yes" active="yes"/>
 <layer number="17" name="Pads" color="2" fill="1" visible="yes" active="yes"/>
@@
 <layer number="28" name="bValues" color="7" fill="1" visible="no" active="yes"/>
 <layer number="29" name="tStop" color="7" fill="3" visible="no" active="yes"/>
-<layer number="30" name="bStop" color="7" fill="6" visible="no" active="yes"/>
+<layer number="30" name="bStop" color="7" fill="6" visible="yes" active="yes"/>
 <layer number="31" name="tCream" color="7" fill="4" visible="no" active="yes"/>
 <layer number="32" name="bCream" color="7" fill="5" visible="no" active="yes"/>
@@
 <attribute name="VALUE" x="22.86" y="0.508" size="0.6096" layer="27" font="vector" ratio="20" align="top-center"/>
 </element>
-<element name="U$1" library="buzzard_labels (5)" package="LED0" value="" x="17.8562" y="9.1948" smashed="yes" rot="MR180"/>
+<element name="U$1" library="buzzard_labels (5)" package="LED0" value="" x="22.5044" y="9.1948" smashed="yes" rot="MR0"/>
 <element name="U$3" library="buzzard_labels" package="SDA5" value="" x="13.97" y="1.4986" smashed="yes" rot="MR90"/>
 <element name="U$10" library="buzzard_labels" package="SCL6" value="" x="16.51" y="1.4986" smashed="yes" rot="MR90"/>
